File: Hardware/Board.brd (EAGLE design)
At the start: 46 x 35 mm, 105 parts, among them IC1 DRV2605YZFR_DRV2605YZFR, IC2 BQ25180YBGR_BQ25180YBGR, IC3 BMA423_BMA423, IC9 RT6160AWSC_RT6160AWSC, J1 503480-2400_503480-2400, J2 TC2030-IDC_TC2030-IDC, J4 KH-TYPE-C-16P_KH-TYPE-C-16P, Q3 ESP32_C6_LIBRARY_6_SI1308EDL-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, U1 NORDIC_NRF_4_NRF52840_QF, U3 ESP32_C6_LIBRARY_MAX17048G+T10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

Commit message: fixed review
Parts:
- moved R17 0.52 mm to (2.92, 8.89)
Routing:
- net N$162: track 0.00 -> 8.30 mm, vias 0 -> 1
- net GND: track 359.8 -> 363.3 mm, vias 5 -> 6
- net N$76: track 41.6 -> 40.9 mm
- added copper zone on layer 1, net GND
- added copper zone on layer 16, net GND
