File: Hardware/Schematic.sch (EAGLE design)
At the start: 105 parts, among them IC1 DRV2605YZFR_DRV2605YZFR, IC2 BQ25180YBGR_BQ25180YBGR, IC3 BMA423_BMA423, IC9 RT6160AWSC_RT6160AWSC, J1 503480-2400_503480-2400, J2 TC2030-IDC_TC2030-IDC, J4 KH-TYPE-C-16P_KH-TYPE-C-16P, Q3 ESP32_C6_LIBRARY_6_SI1308EDL-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, U1 NORDIC_NRF_4_NRF52840_QF, U3 ESP32_C6_LIBRARY_MAX17048G+T10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

Commit message: fixed review
Parts:
- C37: value (none) -> 1uF
- EPD_C10, EPD_C11, EPD_C12, EPD_C5, EPD_C6, EPD_C7, EPD_C8, EPD_C9: value 0.1uF/50V -> 1uF/50V
Connections:
- net N$3 renamed VBUS/2.6D
Other:
- note added: "Q1"
